Commit message: ros stufff

File: rover/urdf/robot.urdf (robot description, URDF)
Before this commit: robot urdf, 2 links, 1 joints
Links:
- removed link rover
- added link base_link; collision mesh filename=package://assets/2020_big.stl; collision mesh filename=package://assets/2020_big.stl
Joints:
- joint Slider 1: parent rover -> base_link
